File: learnboard/learnboard.kicad_pcb (KiCad board)
At the start: 2 copper layers, 281.4 x 146.7 mm, 55 parts, among them SW1 SW_Push, SW10 SW_Push, SW11 SW_Push, SW12 SW_Push, SW13 SW_Push, SW14 SW_Push, SW15 SW_Push, SW16 SW_Push, SW17 RotaryEncoder_Switch_MP, SW2 SW_Push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

Commit message: tried to route things
it is not going very well.
Parts:
- moved D4 237.2 mm to (112.7, 228.2)
- moved D16 165.4 mm to (332.7, 234.7)
- moved D3 19.1 mm to (111.8, 189.8)
- moved A1 2.18 mm to (106.6, 138.9)
- moved D9 0.65 mm to (292.6, 186.9)
Routing:
- net GND: track 0.00 -> 690.0 mm, vias 0 -> 7
- net Col 5: track 0.00 -> 682.1 mm, vias 0 -> 4
- net Row 2: track 0.00 -> 643.4 mm, vias 0 -> 5
- net Col 4: track 0.00 -> 454.9 mm
- net Col 7: track 0.00 -> 453.1 mm
- net Row 1: track 0.00 -> 356.3 mm
- net Net-(D18-A): track 0.00 -> 314.3 mm, vias 0 -> 2
- net Net-(D24-A): track 0.00 -> 310.9 mm
- net Col 8: track 0.00 -> 286.1 mm, vias 0 -> 3
- net Col 2: track 0.00 -> 246.6 mm, vias 0 -> 2
- net Col 6: track 0.00 -> 239.1 mm, vias 0 -> 3
- net Net-(D25-A): track 0.00 -> 238.6 mm
- net Col 1: track 0.00 -> 235.3 mm, vias 0 -> 3
- net DIN: track 0.00 -> 223.0 mm, vias 0 -> 6
- net Net-(D17-A): track 0.00 -> 219.7 mm, vias 0 -> 2
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
Commit message: Fixed lots of DRC errors and added mounting holes
Parts:
- added H1: 5.326mm, MountingHole:MountingHole_5.5mm, F.Cu at (354.0, 134.0)
- added H2: 5.326mm, MountingHole:MountingHole_5.5mm, F.Cu at (144.2, 175.2)
- added H3: 5.326mm, MountingHole:MountingHole_5.5mm, F.Cu at (297.8, 242.5)
- added H4: 5.326mm, MountingHole:MountingHole_5.5mm, F.Cu at (88.0, 244.8)
Routing:
- net GND: track 690.0 -> 766.1 mm, vias 7 -> 10
- net +3V3: track 192.7 -> 216.1 mm, vias 1 -> 2
- net LED 3: track 61.0 -> 76.2 mm, vias 0 -> 3
- net LED 1: track 72.3 -> 86.3 mm, vias 0 -> 2
- net Col 4: track 454.9 -> 465.6 mm, vias 0 -> 1
- net DIN: track 223.0 -> 232.9 mm, vias 6 -> 7
- net Col 2: track 246.6 -> 252.3 mm, vias 2 -> 3
- net Row 2: track 643.4 -> 648.8 mm, vias 5 -> 6
- net LED 7: track 58.4 -> 63.0 mm
- net Col 1: track 235.3 -> 238.6 mm
- net LED 4: track 50.8 -> 53.6 mm
- net Col 8: track 286.1 -> 288.4 mm
- net LED 9: track 73.7 -> 76.0 mm
- net LED 6: track 47.4 -> 49.7 mm
- net LED 10: track 78.1 -> 80.2 mm, vias 1 -> 0
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- added copper zone on B.Cu, net GND
- added copper zone on F.Cu, net GND
Other:
- board size 281.4 x 146.7 mm -> 281.4 x 126 mm
