File: learnboard/learnboard.kicad_pcb (KiCad board)
At the start: 2 copper layers, 281.4 x 126 mm, 59 parts, among them SW1 SW_Push, SW10 SW_Push, SW11 SW_Push, SW12 SW_Push, SW13 SW_Push, SW14 SW_Push, SW15 SW_Push, SW16 SW_Push, SW17 RotaryEncoder_Switch_MP, SW2 SW_Push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

Commit message: Worked on firmware and webapp
Parts:
- D1, D10, D11, D12, D13, D14, D15, D16, D2, D3, D4, D5, D6, D7, D8, D9: footprint Diode_SMD:D_0201_0603Metric_Pad0.64x0.40mm_HandSolder -> Diode_SMD:D_0201_0603Metric
Connections:
- A1 pad 26: unconnected-(A1-GPIO20-Pad26) -> High
- A1 pad 27: unconnected-(A1-GPIO21-Pad27) -> Low
Routing:
- net High: track 0.00 -> 182.2 mm, vias 0 -> 2
- net Low: track 0.00 -> 177.2 mm, vias 0 -> 1
