File: PCB/learnboard.kicad_sch (KiCad schematic)
At the start: 55 parts, among them SW1 SW_Push, SW10 SW_Push, SW11 SW_Push, SW12 SW_Push, SW13 SW_Push, SW14 SW_Push, SW15 SW_Push, SW16 SW_Push, SW17 RotaryEncoder_Switch_MP, SW2 SW_Push, SW3 SW_Push, SW4 SW_Push, SW5 SW_Push, SW6 SW_Push, SW7 SW_Push, SW8 SW_Push, SW9 SW_Push, U1 PCM5100

Commit message: Journalled
Parts:
- U1: footprint Package_CSP:Nexperia_WLCSP-15_2.37x1.17mm_Layout6x3_P0.4mmP0.8mm -> PCM5100APWR:SOP65P640X120-20N
Changed lines of the file:
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@@
 			)
 		)
-		(property "Footprint" "Package_CSP:Nexperia_WLCSP-15_2.37x1.17mm_Layout6x3_P0.4mmP0.8mm"
+		(property "Footprint" "PCM5100APWR:SOP65P640X120-20N"
 			(at 49.53 144.78 0)
 			(hide yes)
